File: bikePump.kicad_pcb (KiCad board)
At the start: 2 copper layers, 19 parts, among them J1 Regulator_2, J2 Regulator_1, J3 Power_In, J4 LCD_Screen, J5 pressure_sensor, Q1 Q_NPN_BCE, Q2 Q_NPN_BCE, SW1 Button_1, SW2 Button_2, SW3 Button_3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

Commit message: updates
Routing:
- net Net-(A1-Pad9): track 72.7 -> 79.2 mm
- net Net-(A1-Pad13): track 40.2 -> 46.7 mm
- net Net-(A1-Pad10): track 82.1 -> 88.6 mm
- net GND: track 0.00 -> 5.01 mm, vias 0 -> 2
- net Net-(A1-Pad27): track 28.7 -> 29.1 mm, vias 1 -> 2
Other:
- board outline added: 101.6 x 85.1 mm
- board text added: "+ -"
- board text added: "A+"
- board text added: "A-"
- board text added: "A0"
- board text added: "A1"
- board text added: "Arduino Nano"
- board text added: "Bike Pump V1 March 23"
- board text added: "GND"
- board text added: "VIN"

Commit message: Updated more of the silkscreen
Parts:
- J4: LCD 1602 : renamed from J4
- J5: Pressure Sensor: renamed from J5
Other:
- board text added: "Adafruit ADS1115"
- board text added: "Pin: 10"
- board text added: "Pin: 6"
- board text added: "Pin: 7"
- board text added: "Pin: A3"
- board text added: "Pin: A6"
- board text added: "Pin: A7"
Changed lines of the file:
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@@
     (property "Sheetname" "")
     (attr through_hole)
-    (fp_text reference "J4" (at 58.452 16.288 unlocked) (layer "F.SilkS")
+    (fp_text reference "J4: LCD 1602 " (at 45.244 16.288 unlocked) (layer "F.SilkS")
       (effects (font (size 4 4) (thickness 0.15)))
     )
     (fp_text value "LCD_Screen" (at 37.465 34.29 unlocked) (layer "F.Fab")
-      (effects (font (size 1 1) (thickness 0.15)))
-    )
-    (fp_text user "${REFERENCE}" (at 38.1 37.465 unlocked) (layer "F.Fab")
       (effects (font (size 1 1) (thickness 0.15)))
     )
@@
       (effects (font (size 1 1) (thickness 0.15)))
     )
-    (fp_text value "Button_1" (at 3.75 6.7) (layer "F.Fab")
+    (fp_text value "Button_1" (at 3.75 6.7) (layer "F.Fab") hide
       (effects (font (size 1 1) (thickness 0.15)))
     )
@@
     (property "Sheetname" "")
     (attr exclude_from_pos_files)
-    (fp_text reference "J5" (at 5.207 -2.413 90) (layer "F.SilkS")
+    (fp_text reference "J5: Pressure Sensor" (at 5.207 -2.413 90) (layer "F.SilkS")
       (effects (font (size 1 1) (thickness 0.15)))
     )
@@
       (effects (font (size 1 1) (thickness 0.15)))
     )
-    (fp_text value "Button_2" (at 2.869 -2.449) (layer "F.Fab")
+    (fp_text value "Button_2" (at 2.869 -2.449) (layer "F.Fab") hide
       (effects (font (size 1 1) (thickness 0.15)))
     )
@@
   (gr_circle (center 161.925 41.275) (end 163.933046 41.275) (layer "Edge.Cuts") (width 0.2) (fill none))
   (gr_rect (start 63.5 38.1) (end 165.1 123.19) (layer "Edge.Cuts") (width 0.2) (fill none))
+  (gr_text "Pin: A3" (at 101.092 111.76) (layer "F.SilkS")
+    (effects (font (size 1 1) (thickness 0.15)))
+  )
   (gr_text "Bike Pump V1\nMarch 23" (at 149.352 83.82 90) (layer "F.SilkS")
     (effects (font (size 2.5 2.5) (thickness 0.15)))
@@
     (effects (font (size 1.5 1.5) (thickness 0.3)))
   )
+  (gr_text "Pin: 7" (at 154.432 39.116) (layer "F.SilkS")
+    (effects (font (size 1 1) (thickness 0.15)))
+  )
+  (gr_text "Adafruit ADS1115" (at 132.08 80.772) (layer "F.SilkS")
+    (effects (font (size 1.5 1.5) (thickness 0.15)))
+  )
   (gr_text "A+" (at 71.12 96.52) (layer "F.SilkS")
     (effects (font (size 1.5 1.5) (thickness 0.3)))
@@
     (effects (font (size 1.5 1.5) (thickness 0.3)))
   )
+  (gr_text "Pin: A6" (at 127.508 111.76) (layer "F.SilkS")
+    (effects (font (size 1 1) (thickness 0.15)))
+  )
+  (gr_text "Pin: A7" (at 153.416 111.76) (layer "F.SilkS")
+    (effects (font (size 1 1) (thickness 0.15)))
+  )
+  (gr_text "Pin: 10" (at 74.676 111.76) (layer "F.SilkS")
+    (effects (font (size 1 1) (thickness 0.15)))
+  )
   (gr_text "GND" (at 127.508 85.344 90) (layer "F.SilkS")
     (effects (font (size 1.5 1.5) (thickness 0.3)))
   )
+  (gr_text "Pin: 6" (at 154.432 61.976) (layer "F.SilkS")
+    (effects (font (size 1 1) (thickness 0.15)))
+  )
   (gr_text "Arduino Nano" (at 86.36 82.804) (layer "F.SilkS")

Commit message: Updates
Parts:
- removed J5: Pressure Sensor: pressure_sensor, Connector_Wire:SolderWire-0.1sqmm_1x04_P3.6mm_D0.4mm_OD1mm
- removed R1, R3: R, Resistor_THT:R_Axial_DIN0207_L6.3mm_D2.5mm_P10.16mm_Horizontal
- added J5: pressure_sensor, Connector_Wire:SolderWire-0.25sqmm_1x04_P4.5mm_D0.65mm_OD2mm, F.Cu at (81.1, 101.6)
- A1: value Arduino_Nano_Every -> Arduino_Nano
- J1, J2, J3: footprint Connector_Wire:SolderWire-0.1sqmm_1x02_P3.6mm_D0.4mm_OD1mm -> Connector_Wire:SolderWire-0.5sqmm_1x02_P4.6mm_D0.9mm_OD2.1mm
- LCD 1602: renamed from J4: LCD 1602 
- U1: value ADS1115_Breakout_board -> AdaFruit_ADS1115
- moved R4 49.9 mm to (146.3, 89.4), turned to 90 degrees
- moved R2 41.1 mm to (138.7, 89.4), turned to 90 degrees
- moved Q2 30.1 mm to (146.2, 95.5), turned to 0 degrees
- moved U1 12.4 mm to (121.4, 89.9), turned to 90 degrees
- moved Q1 9.52 mm to (136.1, 95.5), turned to 0 degrees
- moved SW2 5.97 mm to (151.0, 47.5)
- moved A1 4.07 mm to (107.4, 78.8)
- moved J3 1.45 mm to (160.5, 103.1)
- moved J1 1.15 mm to (160.5, 84.3)
- moved J2 0.44 mm to (160.5, 94.0)
Connections:
- J1 pad 2: Net-(J1-Pad2) -> Net-(Q1-Pad2)
- Q2 pad 2: Net-(Q2-Pad2) -> Net-(J2-Pad2)
Routing:
- net Net-(J5-Pad4): track 78.4 -> 22.6 mm
- net Net-(J5-Pad3): track 88.3 -> 32.7 mm
- net Net-(J5-Pad2): track 93.5 -> 38.5 mm
- net Net-(J5-Pad1): track 99.4 -> 44.4 mm
- net Net-(A1-Pad20): track 18.7 -> 71.6 mm, vias 0 -> 1
- net Net-(A1-Pad21): track 13.0 -> 60.2 mm, vias 0 -> 1
- net Net-(Q2-Pad2): track 38.9 -> 0.00 mm
- net Net-(Q1-Pad1): track 37.8 -> 6.10 mm
- net Net-(J1-Pad2): track 26.2 -> 0.00 mm
- net Net-(Q1-Pad2): track 15.5 -> 39.6 mm, vias 0 -> 1
- net Net-(A1-Pad25): track 67.5 -> 44.4 mm, vias 0 -> 1
- net Net-(A1-Pad26): track 82.4 -> 68.4 mm, vias 0 -> 1
- net Net-(Q2-Pad1): track 19.2 -> 7.09 mm
- net Net-(A1-Pad27): track 29.1 -> 40.8 mm, vias 2 -> 0
- net Net-(A1-Pad11): track 43.3 -> 53.1 mm, vias 1 -> 0
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Other:
- board text added: "Bike Pump V1.1 March 23"
- board text removed: "Adafruit ADS1115"
- board text removed: "Arduino Nano"
- board text removed: "Bike Pump V1 March 23"
